File: LCSDR.kicad_pcb (KiCad board)
At the start: 2 copper layers, 52 x 14 mm, 12 parts, among them P1 IN, P2 OUT, P3 OUT, P4 IN, P5 CONN_01X01, P6 CONN_01X01, U1 AMS1117S33TR

Commit message: Relese version PCB with CNC files
Parts:
- removed P3: OUT, Pin_Headers:Pin_Header_Straight_1x02_Pitch2.54mm
- removed P4: IN, Pin_Headers:Pin_Header_Straight_1x02_Pitch2.54mm
- added P7: CONN_01X01, Mounting_Holes:MountingHole_2.7mm_M2.5_DIN965_Pad, F.Cu at (73.0, -8.00)
- P1: footprint Pin_Headers:Pin_Header_Straight_1x02_Pitch2.54mm -> Pin_Headers:Pin_Header_Straight_1x03_Pitch2.54mm
- P2: footprint Pin_Headers:Pin_Header_Straight_1x02_Pitch2.54mm -> Pin_Headers:Pin_Header_Straight_1x04_Pitch2.54mm
- moved D1 9.82 mm to (26.4, -11.2)
- moved C1 6.76 mm to (25.8, -4.70)
- moved C2 6.54 mm to (20.0, -4.40)
- moved P2 5.66 mm to (46.7, -10.9)
- moved C4 5.07 mm to (37.2, -6.00)
- moved U1 4.55 mm to (31.6, -7.80)
- moved C3 3.30 mm to (41.4, -6.00)
- moved P6 3.00 mm to (53.0, -8.00)
- moved P1 2.12 mm to (10.5, -5.50), turned to 0 degrees
- moved P5 1.00 mm to (5.00, -8.00)
Connections:
- P1 pad 1: Net-(D1-Pad2) -> Net-(C1-Pad1)
- P2 pad 1: Net-(C3-Pad1) -> GND
- P2 pad 2: GND -> Net-(C3-Pad1)
Routing:
- net GND: track 0.06 -> 24.3 mm
- net Net-(C3-Pad1): track 36.0 -> 30.9 mm
- net Net-(C1-Pad1): track 36.2 -> 31.3 mm
- net Net-(D1-Pad2): track 4.29 -> 3.46 mm
Other:
- board outline removed
- net class Default: trace_width 1 -> 0.4
