File: LCSDR.sch (KiCad schematic (older format))
At the start: 12 parts, among them P1 IN, P2 OUT, P3 OUT, P4 IN, P5 CONN_01X01, P6 CONN_01X01, U1 AMS1117S33TR

Commit message: Relese version PCB with CNC files
Parts:
- removed P1, P4: IN, Pin_Headers:Pin_Header_Straight_1x02_Pitch2.54mm, symbol LCSDR-rescue:CONN_01X02-RESCUE-LCSDR
- removed P2, P3: OUT, Pin_Headers:Pin_Header_Straight_1x02_Pitch2.54mm, symbol LCSDR-rescue:CONN_01X02-RESCUE-LCSDR
- added P1: IN, Pin_Headers:Pin_Header_Straight_1x03_Pitch2.54mm, symbol conn:CONN_01X03
- added P2: OUT, Pin_Headers:Pin_Header_Straight_1x04_Pitch2.54mm, symbol conn:CONN_01X04
- added P7: CONN_01X01, Mounting_Holes:MountingHole_2.7mm_M2.5_DIN965_Pad, symbol LCSDR-rescue:CONN_01X01-RESCUE-LCSDR
Other:
- moved on the sheet: P6
Changed lines of the file:
@@
 encoding utf-8
 Sheet 1 1
-Title "Hermes-Lite"
-Date "2016-02-18"
-Rev "2.0-pre1"
-Comp "SofterHardware"
+Title "LD1117 like voltage regulator"
+Date "2017-12-10"
+Rev "1.02"
+Comp "Hardware"
 Comment1 "Vasyl Kuzmenko"
 Comment2 ""
@@
 $EndComp
 $Comp
-L LCSDR-rescue:CONN_01X02-RESCUE-LCSDR P1
-U 1 1 595CE774
-P 3150 1500
-F 0 "P1" H 3150 1650 50  0000 C CNN
-F 1 "IN" V 3250 1500 50  0000 C CNN
-F 2 "Pin_Headers:Pin_Header_Straight_1x02_Pitch2.54mm" H 3150 1500 50  0001 C CNN
-F 3 "" H 3150 1500 50  0000 C CNN
-	1    3150 1500
-	-1   0    0    -1
-$EndComp
-$Comp
 L LCSDR-rescue:CP1_Small-RESCUE-LCSDR C2
 U 1 1 595E762C
@@
 L LCSDR-rescue:GND-RESCUE-LCSDR #PWR02
 U 1 1 5A0FCD8B
-P 7850 1550
-F 0 "#PWR02" H 7850 1300 50  0001 C CNN
-F 1 "GND" H 7850 1400 50  0001 C CNN
-F 2 "" H 7850 1550 50  0000 C CNN
-F 3 "" H 7850 1550 50  0000 C CNN
-	1    7850 1550
+P 7850 1350
+F 0 "#PWR02" H 7850 1100 50  0001 C CNN
+F 1 "GND" H 7850 1200 50  0001 C CNN
+F 2 "" H 7850 1350 50  0000 C CNN
+F 3 "" H 7850 1350 50  0000 C CNN
+	1    7850 1350
 	0    1    1    0
-$EndComp
-$Comp
-L LCSDR-rescue:CONN_01X02-RESCUE-LCSDR P2
-U 1 1 5A0FBCD4
-P 8050 1500
-F 0 "P2" H 8050 1650 50  0000 C CNN
-F 1 "OUT" V 8150 1500 50  0000 C CNN
-F 2 "Pin_Headers:Pin_Header_Straight_1x02_Pitch2.54mm" H 8050 1500 50  0001 C CNN
-F 3 "" H 8050 1500 50  0000 C CNN
-	1    8050 1500
-	1    0    0    -1
-$EndComp
-$Comp
-L LCSDR-rescue:CONN_01X02-RESCUE-LCSDR P3
-U 1 1 5A100D5D
-P 8050 1900
-F 0 "P3" H 8050 2050 50  0000 C CNN
-F 1 "OUT" V 8150 1900 50  0000 C CNN
-F 2 "Pin_Headers:Pin_Header_Straight_1x02_Pitch2.54mm" H 8050 1900 50  0001 C CNN
-F 3 "" H 8050 1900 50  0000 C CNN
-	1    8050 1900
-	1    0    0    -1
 $EndComp
 $Comp
 L LCSDR-rescue:GND-RESCUE-LCSDR #PWR08
 U 1 1 5A100D8F
-P 7850 1950
-F 0 "#PWR08" H 7850 1700 50  0001 C CNN
-F 1 "GND" H 7850 1800 50  0001 C CNN
-F 2 "" H 7850 1950 50  0000 C CNN
-F 3 "" H 7850 1950 50  0000 C CNN
-	1    7850 1950
+P 7850 1650
+F 0 "#PWR08" H 7850 1400 50  0001 C CNN
+F 1 "GND" H 7850 1500 50  0001 C CNN
+F 2 "" H 7850 1650 50  0000 C CNN
+F 3 "" H 7850 1650 50  0000 C CNN
+	1    7850 1650
 	0    1    1    0
 $EndComp
-Wire Wire Line
-	7850 1850 7700 1850
-Wire Wire Line
-	7700 1850 7700 1450
-Connection ~ 7700 1450
-$Comp
-L LCSDR-rescue:CONN_01X02-RESCUE-LCSDR P4
-U 1 1 5A100E1B
-P 3950 1950
-F 0 "P4" H 3950 2100 50  0000 C CNN
-F 1 "IN" V 4050 1950 50  0000 C CNN
-F 2 "Pin_Headers:Pin_Header_Straight_1x02_Pitch2.54mm" H 3950 1950 50  0001 C CNN
-F 3 "" H 3950 1950 50  0000 C CNN
-	1    3950 1950
-	-1   0    0    -1
-$EndComp
-Wire Wire Line
-	4150 1900 4300 1900
-Wire Wire Line
-	4300 1900 4300 1450
 Connection ~ 4300 1450
-$Comp
-L LCSDR-rescue:GND-RESCUE-LCSDR #PWR09
-U 1 1 5A100E68
-P 4150 2000
-F 0 "#PWR09" H 4150 1750 50  0001 C CNN
-F 1 "GND" H 4150 1850 50  0001 C CNN
-F 2 "" H 4150 2000 50  0000 C CNN
-F 3 "" H 4150 2000 50  0000 C CNN
-	1    4150 2000
-	0    -1   -1   0
-$EndComp
 $Comp
 L LCSDR-rescue:CONN_01X01-RESCUE-LCSDR P6
 U 1 1 5AA9F4A9
-P 8650 1700
-F 0 "P6" H 8727 1786 50  0000 L CNN
-F 1 "CONN_01X01" H 8727 1695 50  0000 L CNN
-F 2 "Mounting_Holes:MountingHole_2.7mm_M2.5_DIN965_Pad" H 8727 1604 50  0000 L CNN
-F 3 "" H 8650 1700 50  0000 C CNN
-	1    8650 1700
+P 8650 2400
+F 0 "P6" H 8727 2486 50  0000 L CNN
+F 1 "CONN_01X01" H 8727 2395 50  0000 L CNN
+F 2 "Mounting_Holes:MountingHole_2.7mm_M2.5_DIN965_Pad" H 8727 2304 50  0000 L CNN
+F 3 "" H 8650 2400 50  0000 C CNN
+	1    8650 2400
 	1    0    0    -1
 $EndComp
@@
 L LCSDR-rescue:GND-RESCUE-LCSDR #PWR010
 U 1 1 5AA9F709
-P 8450 1700
-F 0 "#PWR010" H 8450 1450 50  0001 C CNN
-F 1 "GND" H 8450 1550 50  0001 C CNN
-F 2 "" H 8450 1700 50  0000 C CNN
-F 3 "" H 8450 1700 50  0000 C CNN
-	1    8450 1700
+P 8450 2400
+F 0 "#PWR010" H 8450 2150 50  0001 C CNN
+F 1 "GND" H 8450 2250 50  0001 C CNN
+F 2 "" H 8450 2400 50  0000 C CNN
+F 3 "" H 8450 2400 50  0000 C CNN
+	1    8450 2400
 	0    1    1    0
 $EndComp
@@
 $EndComp
 Wire Wire Line
-	3650 1450 3350 1450
-Wire Wire Line
 	5250 1450 5800 1450
 Wire Wire Line
@@
 	7100 1450 7300 1450
 Wire Wire Line
-	7300 1450 7700 1450
-Wire Wire Line
-	7700 1450 7850 1450
-Wire Wire Line
 	4300 1450 4850 1450
+$Comp
+L LCSDR-rescue:CONN_01X01-RESCUE-LCSDR P7
+U 1 1 5A27AB24
+P 8650 2050
+F 0 "P7" H 8727 2136 50  0000 L CNN
+F 1 "CONN_01X01" H 8727 2045 50  0000 L CNN
+F 2 "Mounting_Holes:MountingHole_2.7mm_M2.5_DIN965_Pad" H 8727 1954 50  0000 L CNN
+F 3 "" H 8650 2050 50  0000 C CNN
+	1    8650 2050
+	1    0    0    -1
+$EndComp
+$Comp
+L LCSDR-rescue:GND-RESCUE-LCSDR #PWR012
+U 1 1 5A27AB2A
+P 8450 2050
+F 0 "#PWR012" H 8450 1800 50  0001 C CNN
+F 1 "GND" H 8450 1900 50  0001 C CNN
+F 2 "" H 8450 2050 50  0000 C CNN
+F 3 "" H 8450 2050 50  0000 C CNN
+	1    8450 2050
+	0    1    1    0
+$EndComp
+$Comp
+L conn:CONN_01X04 P2
+U 1 1 5A27AE8B
+P 8050 1500
+F 0 "P2" H 8128 1541 50  0000 L CNN
+F 1 "OUT" H 8128 1450 50  0000 L CNN
+F 2 "Pin_Headers:Pin_Header_Straight_1x04_Pitch2.54mm" H 8050 1500 50  0001 C CNN
+F 3 "" H 8050 1500 50  0000 C CNN
+	1    8050 1500
+	1    0    0    -1
+$EndComp
+Wire Wire Line
+	7850 1550 7750 1550
+Wire Wire Line
+	7750 1550 7750 1450
+Wire Wire Line
+	7300 1450 7750 1450
+Connection ~ 7750 1450
+Wire Wire Line
+	7750 1450 7850 1450
+$Comp
+L conn:CONN_01X03 P1
+U 1 1 5A27BAF0
+P 3150 1550
+F 0 "P1" H 3069 1225 50  0000 C CNN
+F 1 "IN" H 3069 1316 50  0000 C CNN
+F 2 "Pin_Headers:Pin_Header_Straight_1x03_Pitch2.54mm" H 3150 1550 50  0001 C CNN
+F 3 "" H 3150 1550 50  0000 C CNN
+	1    3150 1550
+	-1   0    0    1
+$EndComp
+Wire Wire Line
+	3350 1450 3650 1450
+Wire Wire Line
+	3350 1650 4300 1650
+Wire Wire Line
+	4300 1650 4300 1450
 $EndSCHEMATC
